File: OS/3.0/AC_driver/acdr_3.2.brd (EAGLE design)
At the start: 100 x 45 mm, 61 parts, among them T1 BT1308W

Commit message: correct the pull down resistor value
Parts:
- RB1, RB2, RB3, RB4, RB5, RB6, RB7, RB8: value 470K -> 10K
Changed lines of the file:
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@@
 <?xml version="1.0" encoding="utf-8"?>
 <!DOCTYPE eagle SYSTEM "eagle.dtd">
-<eagle version="7.1.0">
+<eagle version="9.6.2">
 <drawing>
 <settings>
 <setting alwaysvectorfont="yes"/>
+<setting keepoldvectorfont="yes"/>
 <setting verticaltext="up"/>
 </settings>
@@
 <param name="dpMaxLengthDifference" value="10mm"/>
 <param name="dpGapFactor" value="2.5"/>
-<param name="checkGrid" value="0"/>
 <param name="checkAngle" value="0"/>
 <param name="checkFont" value="1"/>
 <param name="checkRestrict" value="0"/>
+<param name="checkStop" value="0"/>
+<param name="checkValues" value="0"/>
+<param name="checkNames" value="1"/>
+<param name="checkWireStubs" value="1"/>
+<param name="checkPolygonWidth" value="0"/>
 <param name="useDiameter" value="13"/>
 <param name="maxErrors" value="50"/>
@@
 <attribute name="VALUE" x="86.714" y="14.54" size="1.27" layer="27" ratio="10" rot="R270"/>
 </element>
-<element name="RB1" library="rcl" package="R0603" value="470K" x="47" y="28" smashed="yes">
+<element name="RB1" library="rcl" package="R0603" value="10K" x="47" y="28" smashed="yes">
 <attribute name="NAME" x="46" y="29" size="0.8128" layer="25" ratio="15"/>
 <attribute name="VALUE" x="46.365" y="26.095" size="1.27" layer="27"/>
 </element>
-<element name="RB2" library="rcl" package="R0603" value="470K" x="54" y="28" smashed="yes">
+<element name="RB2" library="rcl" package="R0603" value="10K" x="54" y="28" smashed="yes">
 <attribute name="NAME" x="53" y="29" size="0.8128" layer="25" ratio="15"/>
 <attribute name="VALUE" x="53.365" y="26.095" size="1.27" layer="27"/>
 </element>
-<element name="RB3" library="rcl" package="R0603" value="470K" x="61" y="28" smashed="yes">
+<element name="RB3" library="rcl" package="R0603" value="10K" x="61" y="28" smashed="yes">
 <attribute name="NAME" x="60" y="29" size="0.8128" layer="25" ratio="15"/>
 <attribute name="VALUE" x="60.365" y="26.095" size="1.27" layer="27"/>
 </element>
-<element name="RB4" library="rcl" package="R0603" value="470K" x="68" y="28" smashed="yes">
+<element name="RB4" library="rcl" package="R0603" value="10K" x="68" y="28" smashed="yes">
 <attribute name="NAME" x="67" y="29" size="0.8128" layer="25" ratio="15"/>
 <attribute name="VALUE" x="67.365" y="26.095" size="1.27" layer="27"/>
 </element>
-<element name="RB5" library="rcl" package="R0603" value="470K" x="75" y="28" smashed="yes">
+<element name="RB5" library="rcl" package="R0603" value="10K" x="75" y="28" smashed="yes">
 <attribute name="NAME" x="74" y="29" size="0.8128" layer="25" ratio="15"/>
 <attribute name="VALUE" x="74.365" y="26.095" size="1.27" layer="27"/>
 </element>
-<element name="RB6" library="rcl" package="R0603" value="470K" x="82" y="28" smashed="yes">
+<element name="RB6" library="rcl" package="R0603" value="10K" x="82" y="28" smashed="yes">
 <attribute name="NAME" x="81" y="29" size="0.8128" layer="25" ratio="15"/>
 <attribute name="VALUE" x="81.365" y="26.095" size="1.27" layer="27"/>
 </element>
-<element name="RB7" library="rcl" package="R0603" value="470K" x="89" y="28" smashed="yes">
+<element name="RB7" library="rcl" package="R0603" value="10K" x="89" y="28" smashed="yes">
 <attribute name="NAME" x="88" y="29" size="0.8128" layer="25" ratio="15"/>
 <attribute name="VALUE" x="88.365" y="26.095" size="1.27" layer="27"/>
 </element>
-<element name="RB8" library="rcl" package="R0603" value="470K" x="96" y="28" smashed="yes">
+<element name="RB8" library="rcl" package="R0603" value="10K" x="96" y="28" smashed="yes">
 <attribute name="NAME" x="95" y="29" size="0.8128" layer="25" ratio="15"/>
 <attribute name="VALUE" x="95.365" y="26.095" size="1.27" layer="27"/>
@@
 <attribute name="MF" value="" x="52.8" y="33" size="1.778" layer="27" display="off"/>
 <attribute name="MPN" value="" x="52.8" y="33" size="1.778" layer="27" display="off"/>
+<attribute name="NAME" x="48.6275" y="32.67" size="0.8128" layer="25" ratio="15"/>
 <attribute name="OC_FARNELL" value="unknown" x="52.8" y="33" size="1.778" layer="27" display="off"/>
 <attribute name="OC_NEWARK" value="unknown" x="52.8" y="33" size="1.778" layer="27" display="off"/>
-<attribute name="NAME" x="48.6275" y="32.67" size="0.8128" layer="25" ratio="15"/>
 <attribute name="VALUE" x="50.8275" y="30.46" size="1.27" layer="27"/>
 </element>
@@
 <attribute name="MF" value="" x="56.5" y="33" size="1.778" layer="27" display="off"/>
 <attribute name="MPN" value="" x="56.5" y="33" size="1.778" layer="27" display="off"/>
+<attribute name="NAME" x="58.6275" y="32.77" size="0.8128" layer="25" ratio="15"/>
 <attribute name="OC_FARNELL" value="unknown" x="56.5" y="33" size="1.778" layer="27" display="off"/>
 <attribute name="OC_NEWARK" value="unknown" x="56.5" y="33" size="1.778" layer="27" display="off"/>
-<attribute name="NAME" x="58.6275" y="32.77" size="0.8128" layer="25" ratio="15"/>
 <attribute name="VALUE" x="54.5275" y="30.46" size="1.27" layer="27"/>
 </element>
@@
 </element>
 <element name="1509" library="adafruit" package="SO08" value="34063" x="30.775" y="14" smashed="yes" rot="R270">
+<attribute name="NAME" x="30.421" y="15.33" size="0.8128" layer="25" ratio="15" rot="SR270"/>
 <attribute name="VALUE" x="28.743" y="10.063" size="1.27" layer="27" ratio="10"/>
-<attribute name="NAME" x="30.421" y="15.33" size="0.8128" layer="25" ratio="15" rot="SR270"/>
 </element>
 <element name="RS1" library="adafruit2013" package="R0603" value="4K7" x="28" y="8.5" smashed="yes">
@@
 </signal>
 </signals>
+<mfgpreviewcolors>
+<mfgpreviewcolor name="soldermaskcolor" color="0xC8008000"/>
+<mfgpreviewcolor name="silkscreencolor" color="0xFFFEFEFE"/>
+<mfgpreviewcolor name="backgroundcolor" color="0xFF282828"/>
+<mfgpreviewcolor name="coppercolor" color="0xFFFFBF00"/>
+<mfgpreviewcolor name="substratecolor" color="0xFF786E46"/>
+</mfgpreviewcolors>
 <errors>
 </errors>
