File: OS/3.0/DC_driver/dcdr_3.2.brd (EAGLE design)
At the start: 100 x 45 mm, 75 parts, among them T1 AO3400, T2 AO3400, T3 AO3400, T4 AO3400, T5 AO3400, T6 AO3400, T7 AO3400, T8 AO3400

Commit message: correcting os3.2 dc driver part number
Parts:
- QB1, QB2: value MMBT3904 -> AO3400
- RV1, RV2: value 1K -> 10K
Changed lines of the file:
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@@
 <?xml version="1.0" encoding="utf-8"?>
 <!DOCTYPE eagle SYSTEM "eagle.dtd">
-<eagle version="7.1.0">
+<eagle version="9.6.2">
 <drawing>
 <settings>
 <setting alwaysvectorfont="yes"/>
+<setting keepoldvectorfont="yes"/>
 <setting verticaltext="up"/>
 </settings>
@@
 <param name="dpMaxLengthDifference" value="10mm"/>
 <param name="dpGapFactor" value="2.5"/>
-<param name="checkGrid" value="0"/>
 <param name="checkAngle" value="0"/>
 <param name="checkFont" value="1"/>
 <param name="checkRestrict" value="0"/>
+<param name="checkStop" value="0"/>
+<param name="checkValues" value="0"/>
+<param name="checkNames" value="1"/>
+<param name="checkWireStubs" value="1"/>
+<param name="checkPolygonWidth" value="0"/>
 <param name="useDiameter" value="13"/>
 <param name="maxErrors" value="50"/>
@@
 <attribute name="VALUE" x="22.595" y="22.825" size="1.27" layer="27"/>
 </element>
-<element name="QB1" library="SparkFunNew" package="SOT23-3" value="MMBT3904" x="25" y="18.5" smashed="yes" rot="R90">
+<element name="QB1" library="SparkFunNew" package="SOT23-3" value="AO3400" x="25" y="18.5" smashed="yes" rot="R90">
 <attribute name="NAME" x="23" y="17.5" size="0.8128" layer="25" ratio="15" rot="R90"/>
 <attribute name="VALUE" x="25.1905" y="17.484" size="0.4064" layer="27" rot="R90"/>
@@
 <attribute name="VALUE" x="33.595" y="16.825" size="1.27" layer="27"/>
 </element>
-<element name="QB2" library="SparkFunNew" package="SOT23-3" value="MMBT3904" x="40.5" y="15.5" smashed="yes" rot="R90">
+<element name="QB2" library="SparkFunNew" package="SOT23-3" value="AO3400" x="40.5" y="15.5" smashed="yes" rot="R90">
 <attribute name="NAME" x="38.5" y="14.5" size="0.8128" layer="25" ratio="15" rot="R90"/>
 <attribute name="VALUE" x="40.6905" y="14.484" size="0.4064" layer="27" rot="R90"/>
@@
 <attribute name="VALUE" x="32.889" y="8.532" size="1.27" layer="27" rot="R180"/>
 </element>
-<element name="RV1" library="adafruitGood" package="R0603" value="1K" x="28" y="18.5" smashed="yes" rot="R270">
+<element name="RV1" library="adafruitGood" package="R0603" value="10K" x="28" y="18.5" smashed="yes" rot="R270">
 <attribute name="NAME" x="28.889" y="19.389" size="0.8128" layer="25" rot="R270"/>
 <attribute name="VALUE" x="25.968" y="19.389" size="1.27" layer="27" rot="R270"/>
 </element>
-<element name="RV2" library="adafruitGood" package="R0603" value="1K" x="43.5" y="15.5" smashed="yes" rot="R270">
+<element name="RV2" library="adafruitGood" package="R0603" value="10K" x="43.5" y="15.5" smashed="yes" rot="R270">
 <attribute name="NAME" x="44.389" y="16.489" size="0.8128" layer="25" rot="R270"/>
 <attribute name="VALUE" x="41.468" y="16.389" size="1.27" layer="27" rot="R270"/>
@@
 </signal>
 </signals>
+<mfgpreviewcolors>
+<mfgpreviewcolor name="soldermaskcolor" color="0xC8008000"/>
+<mfgpreviewcolor name="silkscreencolor" color="0xFFFEFEFE"/>
+<mfgpreviewcolor name="backgroundcolor" color="0xFF282828"/>
+<mfgpreviewcolor name="coppercolor" color="0xFFFFBF00"/>
+<mfgpreviewcolor name="substratecolor" color="0xFF786E46"/>
+</mfgpreviewcolors>
 <errors>
 </errors>
