File: OSPi/1.52/ospi152.brd (EAGLE design)
At the start: 100 x 80 mm, 70 parts, among them J0 ACIN, T1 Z0103MN, T2 Z0103MN, T3 Z0103MN, T4 Z0103MN, T5 Z0103MN, T6 Z0103MN, T7 Z0103MN, T8 Z0103MN

Commit message: add OS3.3 master board design files
Parts:
- CS1, CS2, CS3, CS4, CS5, CS6, CS7, CS8: value 0.1u -> 0.01u
Changed lines of the file:
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@@
 <setting verticaltext="up"/>
 </settings>
-<grid distance="0.5" unitdist="mm" unit="mm" style="dots" multiple="1" display="yes" altdistance="0.01" altunitdist="inch" altunit="inch"/>
+<grid distance="0.05" unitdist="mm" unit="mm" style="dots" multiple="1" display="yes" altdistance="0.01" altunitdist="inch" altunit="inch"/>
 <layers>
 <layer number="1" name="Top" color="4" fill="1" visible="yes" active="yes"/>
@@
 <text x="34.5" y="18" size="1.016" layer="21" ratio="15">RPi Pin Headers</text>
 <text x="65.5" y="65" size="1.27" layer="21" font="vector" ratio="15" rot="SR180">(obsolete)</text>
+<circle x="3" y="4" radius="3" width="0" layer="42"/>
+<circle x="97" y="4" radius="3" width="0" layer="42"/>
+<circle x="3" y="76" radius="3" width="0" layer="42"/>
+<circle x="97" y="76" radius="3" width="0" layer="42"/>
 </plain>
 <attributes>
@@
 <attribute name="VALUE" x="28.532" y="20.611" size="1.27" layer="27" rot="R90"/>
 </element>
-<element name="CS1" library="adafruit" package="C0603K" value="0.1u" x="26.5" y="24.5" smashed="yes" rot="R90">
+<element name="CS1" library="adafruit" package="C0603K" value="0.01u" x="26.5" y="24.5" smashed="yes" rot="R90">
 <attribute name="VALUE" x="28.15" y="23.7" size="1.016" layer="27" rot="R90"/>
 </element>
@@
 <attribute name="VALUE" x="35.532" y="20.611" size="1.27" layer="27" rot="R90"/>
 </element>
-<element name="CS2" library="adafruit" package="C0603K" value="0.1u" x="33.5" y="24.5" smashed="yes" rot="R90">
+<element name="CS2" library="adafruit" package="C0603K" value="0.01u" x="33.5" y="24.5" smashed="yes" rot="R90">
 <attribute name="VALUE" x="35.15" y="23.7" size="1.016" layer="27" rot="R90"/>
 </element>
@@
 <attribute name="VALUE" x="42.532" y="20.611" size="1.27" layer="27" rot="R90"/>
 </element>
-<element name="CS3" library="adafruit" package="C0603K" value="0.1u" x="40.5" y="24.5" smashed="yes" rot="R90">
+<element name="CS3" library="adafruit" package="C0603K" value="0.01u" x="40.5" y="24.5" smashed="yes" rot="R90">
 <attribute name="VALUE" x="42.15" y="23.7" size="1.016" layer="27" rot="R90"/>
 </element>
@@
 <attribute name="VALUE" x="49.532" y="20.611" size="1.27" layer="27" rot="R90"/>
 </element>
-<element name="CS4" library="adafruit" package="C0603K" value="0.1u" x="47.5" y="24.5" smashed="yes" rot="R90">
+<element name="CS4" library="adafruit" package="C0603K" value="0.01u" x="47.5" y="24.5" smashed="yes" rot="R90">
 <attribute name="VALUE" x="49.15" y="23.7" size="1.016" layer="27" rot="R90"/>
 </element>
@@
 <attribute name="VALUE" x="56.532" y="20.611" size="1.27" layer="27" rot="R90"/>
 </element>
-<element name="CS5" library="adafruit" package="C0603K" value="0.1u" x="54.5" y="24.5" smashed="yes" rot="R90">
+<element name="CS5" library="adafruit" package="C0603K" value="0.01u" x="54.5" y="24.5" smashed="yes" rot="R90">
 <attribute name="VALUE" x="56.15" y="23.7" size="1.016" layer="27" rot="R90"/>
 </element>
@@
 <attribute name="VALUE" x="63.532" y="20.611" size="1.27" layer="27" rot="R90"/>
 </element>
-<element name="CS6" library="adafruit" package="C0603K" value="0.1u" x="61.5" y="24.5" smashed="yes" rot="R90">
+<element name="CS6" library="adafruit" package="C0603K" value="0.01u" x="61.5" y="24.5" smashed="yes" rot="R90">
 <attribute name="VALUE" x="63.15" y="23.7" size="1.016" layer="27" rot="R90"/>
 </element>
@@
 <attribute name="VALUE" x="70.532" y="20.611" size="1.27" layer="27" rot="R90"/>
 </element>
-<element name="CS7" library="adafruit" package="C0603K" value="0.1u" x="68.5" y="24.5" smashed="yes" rot="R90">
+<element name="CS7" library="adafruit" package="C0603K" value="0.01u" x="68.5" y="24.5" smashed="yes" rot="R90">
 <attribute name="VALUE" x="70.15" y="23.7" size="1.016" layer="27" rot="R90"/>
 </element>
@@
 <attribute name="VALUE" x="77.532" y="20.611" size="1.27" layer="27" rot="R90"/>
 </element>
-<element name="CS8" library="adafruit" package="C0603K" value="0.1u" x="75.5" y="24.5" smashed="yes" rot="R90">
+<element name="CS8" library="adafruit" package="C0603K" value="0.01u" x="75.5" y="24.5" smashed="yes" rot="R90">
 <attribute name="VALUE" x="77.15" y="23.7" size="1.016" layer="27" rot="R90"/>
 </element>
@@
 <wire x1="8.98128125" y1="68.918715625" x2="6.031284375" y2="68.918715625" width="0.8128" layer="1"/>
 <wire x1="6.031284375" y1="68.918715625" x2="5" y2="69.95" width="0.8128" layer="1"/>
-<wire x1="3.722" y1="64.5" x2="3.722" y2="73.422" width="0.8128" layer="16"/>
-<wire x1="8.07" y1="77.77" x2="3.722" y2="73.422" width="0.8128" layer="16"/>
-<wire x1="8.07" y1="77.77" x2="9.87" y2="77.77" width="0.8128" layer="16"/>
+<wire x1="3.722" y1="70.172" x2="3.722" y2="64.5" width="0.8128" layer="16"/>
 <wire x1="9.87" y1="77.77" x2="12.41" y2="77.77" width="0.8128" layer="1"/>
 <wire x1="17.095" y1="47.9266" x2="17.095" y2="49.395" width="0.6096" layer="1"/>
@@
 <wire x1="91.9" y1="11.5" x2="78.4" y2="11.5" width="0.3048" layer="1"/>
 <wire x1="76.7" y1="65.7" x2="77.9" y2="66.9" width="0.3048" layer="1"/>
+<wire x1="9.87" y1="77.77" x2="8.72" y2="77.77" width="0.8128" layer="16"/>
+<wire x1="8.72" y1="77.77" x2="7.65" y2="76.7" width="0.8128" layer="16"/>
+<wire x1="7.65" y1="74.1" x2="3.722" y2="70.172" width="0.8128" layer="16"/>
+<wire x1="7.65" y1="76.7" x2="7.65" y2="74.1" width="0.8128" layer="16"/>
 </signal>
 <signal name="N$4">
@@
 <mfgpreviewcolor name="substratecolor" color="0xFF786E46"/>
 </mfgpreviewcolors>
-<errors>
-</errors>
 </board>
 </drawing>
