File: OSPi/1.52/ospi152.sch (EAGLE design)
At the start: 70 parts, among them J0 ACIN, T1 Z0103MN, T2 Z0103MN, T3 Z0103MN, T4 Z0103MN, T5 Z0103MN, T6 Z0103MN, T7 Z0103MN, T8 Z0103MN

Commit message: add OS3.3 master board design files
Parts:
- CS1, CS2, CS3, CS4, CS5, CS6, CS7, CS8: value 0.1u -> 0.01u
Changed lines of the file:
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@@
 <part name="P+2" library="supply1" deviceset="VCC" device=""/>
 <part name="RS1" library="adafruit2013" deviceset="R-US_" device="R0603" value="47"/>
-<part name="CS1" library="adafruit" deviceset="C-US" device="C0603K" value="0.1u"/>
+<part name="CS1" library="adafruit" deviceset="C-US" device="C0603K" value="0.01u"/>
 <part name="RS2" library="adafruit2013" deviceset="R-US_" device="R0603" value="47"/>
-<part name="CS2" library="adafruit" deviceset="C-US" device="C0603K" value="0.1u"/>
+<part name="CS2" library="adafruit" deviceset="C-US" device="C0603K" value="0.01u"/>
 <part name="RS3" library="adafruit2013" deviceset="R-US_" device="R0603" value="47"/>
-<part name="CS3" library="adafruit" deviceset="C-US" device="C0603K" value="0.1u"/>
+<part name="CS3" library="adafruit" deviceset="C-US" device="C0603K" value="0.01u"/>
 <part name="RS4" library="adafruit2013" deviceset="R-US_" device="R0603" value="47"/>
-<part name="CS4" library="adafruit" deviceset="C-US" device="C0603K" value="0.1u"/>
+<part name="CS4" library="adafruit" deviceset="C-US" device="C0603K" value="0.01u"/>
 <part name="RS5" library="adafruit2013" deviceset="R-US_" device="R0603" value="47"/>
-<part name="CS5" library="adafruit" deviceset="C-US" device="C0603K" value="0.1u"/>
+<part name="CS5" library="adafruit" deviceset="C-US" device="C0603K" value="0.01u"/>
 <part name="RS6" library="adafruit2013" deviceset="R-US_" device="R0603" value="47"/>
-<part name="CS6" library="adafruit" deviceset="C-US" device="C0603K" value="0.1u"/>
+<part name="CS6" library="adafruit" deviceset="C-US" device="C0603K" value="0.01u"/>
 <part name="RS7" library="adafruit2013" deviceset="R-US_" device="R0603" value="47"/>
-<part name="CS7" library="adafruit" deviceset="C-US" device="C0603K" value="0.1u"/>
+<part name="CS7" library="adafruit" deviceset="C-US" device="C0603K" value="0.01u"/>
 <part name="RS8" library="adafruit2013" deviceset="R-US_" device="R0603" value="47"/>
-<part name="CS8" library="adafruit" deviceset="C-US" device="C0603K" value="0.1u"/>
+<part name="CS8" library="adafruit" deviceset="C-US" device="C0603K" value="0.01u"/>
 <part name="XL2011" library="adafruit" deviceset="XL2001" device="" value="XL2011"/>
 <part name="C4" library="adafruit" deviceset="C-US" device="C0603K" value="105"/>
